File: pcb.kicad_pcb (KiCad board)
At the start: 2 copper layers, 53.3 x 152.4 mm, 21 parts, among them J2 3vJumper1, J3 3vJumper1, SW1 RotaryEncoder_Switch_MP, U1 LM1117T-3.3

Commit message: updated to support both c3 mini and a c3/S3 zero
Parts:
- added J4: 3vJumper1, Connector_PinHeader_2.54mm:PinHeader_1x01_P2.54mm_Vertical, F.Cu at (108.2, 127.9)
- D1: value SR2002 R0 (500ma 20V) -> 1N5819
- MCU1: value ESP32S3Zero -> ESP32 C3 Mini
- USB1: value USB -> USB Conn
Connections:
- MCU1 pad 16: unconnected-(C2-D13-Pad16) -> /ROT_CLK
- MCU1 pad 9: /ROT_CLK -> unconnected-(MCU1-D6-Pad9)
Routing:
- net /ROT_CLK: track 23.5 -> 36.0 mm
- net unconnected-(MCU1-D6-Pad9): track 0.00 -> 2.77 mm
